File: pcb/open-vaporphase/open-vaporphase.kicad_sch (KiCad schematic)
At the start: 9 parts, among them J1 USB_C_Receptacle, J2 Conn_01x02_Pin, SW1 SW_Push, U1 ESP32-S3-WROOM-1

Commit message: schematic wip
Signed-off-by: 3nt3 <gott@3nt3.de>
Parts:
- added J3: Conn_01x03_Socket, symbol Connector:Conn_01x03_Socket
Connections:
- net GND: now also J3.3 (Pin_3)
- net FUSE_ACTIVATED: now reaches U1.12 (GPIO8/TOUCH8/ADC1_CH7/SUBSPICS1)
- net I2C_CLK: no longer names the net of U1.7 (GPIO7/TOUCH7/ADC1_CH6)
- net I2C_CLK: now also J3.2 (Pin_2)
- net I2C_SDA: no longer names the net of U1.6 (GPIO6/TOUCH6/ADC1_CH5)
- net I2C_SDA: now also J3.1 (Pin_1)
- no-connect marks 0 -> 10
Other:
- moved on the sheet: C1, C2, C3, J2, SW1, U1
